File: big/Glup-big.kicad_pcb (KiCad board)
At the start: 2 copper layers, 174.6 x 109.5 mm, 50 parts, among them J2 MJ-4PP-9, SW1 SW_PUSH, SW10 SW_PUSH, SW11 SW_PUSH, SW12 SW_PUSH, SW13 SW_PUSH, SW14 SW_PUSH, SW15 SW_PUSH, SW16 SW_PUSH, SW17 SW_PUSH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

Commit message: separate big and little glup
Other:
- board size 174.6 x 109.5 mm -> 145.7 x 109.5 mm
Changed lines of the file:
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@@
   (gr_line (start 168.795342 40.977298) (end 189.06 40.94)
     (stroke (width 0.1) (type default)) (layer "Edge.Cuts"))
-  (gr_line (start 216.923999 120.973) (end 216.923999 113.723)
-    (stroke (width 0.15) (type solid)) (layer "Edge.Cuts"))
-  (gr_line (start 216.916 49.599) (end 216.916 42.349)
-    (stroke (width 0.15) (type solid)) (layer "Edge.Cuts"))
   (gr_line (start 189.06 40.94) (end 189.08 103.91)
     (stroke (width 0.1) (type default)) (layer "Edge.Cuts"))
-  (gr_line (start 217.916 42.349) (end 217.916 49.599)
-    (stroke (width 0.15) (type solid)) (layer "Edge.Cuts"))
-  (gr_arc (start 66.703999 133.965) (mid 67.057552 134.111447) (end 67.203999 134.465)
-    (stroke (width 0.15) (type solid)) (layer "Edge.Cuts"))
   (gr_line (start 170.04 136.59) (end 189.08 103.91)
     (stroke (width 0.1) (type default)) (layer "Edge.Cuts"))
   (gr_line (start 109.81 120.34) (end 130.81 120.34)
     (stroke (width 0.1) (type default)) (layer "Edge.Cuts"))
-  (gr_line (start 217.923999 113.723) (end 217.923999 120.973)
-    (stroke (width 0.15) (type solid)) (layer "Edge.Cuts"))
   (gr_arc (start 116.917513 27.099036) (mid 143.742599 30.725601) (end 168.795342 40.977298)
     (stroke (width 0.1) (type default)) (layer "Edge.Cuts"))
@@
   (gr_line (start 43.35 61.68) (end 43.41 120.39)
     (stroke (width 0.1) (type default)) (layer "Edge.Cuts"))
-  (gr_arc (start 66.203999 134.465) (mid 66.350446 134.111447) (end 66.703999 133.965)
-    (stroke (width 0.15) (type solid)) (layer "Edge.Cuts"))
-  (gr_arc (start 217.916 49.599) (mid 217.769553 49.952553) (end 217.416 50.099)
-    (stroke (width 0.15) (type solid)) (layer "Edge.Cuts"))
   (gr_line (start 43.41 120.39) (end 109.81 120.34)
     (stroke (width 0.1) (type default)) (layer "Edge.Cuts"))
   (gr_line (start 151.47 125.89) (end 170.04 136.59)
     (stroke (width 0.1) (type default)) (layer "Edge.Cuts"))
-  (gr_arc (start 217.416 50.099) (mid 217.062447 49.952553) (end 216.916 49.599)
-    (stroke (width 0.15) (type solid)) (layer "Edge.Cuts"))
   (gr_line (start 130.81 120.34) (end 151.47 125.89)
     (stroke (width 0.1) (type default)) (layer "Edge.Cuts"))
